File: eagle/encoder_board.sch (EAGLE design)
At the start: 166 parts, among them CN1 6p-2.54, IC1 MEGA8-MI, IC2 AT42QT1010SOT23, X1 52745-0690, X2 52745-0690, X3 52745-0690, X4 POGOPIN-CONNWITHVIAS-SMV, X5 52745-0690

Commit message: Divide boards in design to separate files
Parts:
- removed C1, C10, C11, C12, C13, C14, C15, C2, C20, C21, C22, C24, C3, C4, C41, C42, C43, C44, C45, C46, C47, C48, C49, C5, C50, C51, C52, C53, C54, C55, C6, C7, C8, C9: 100n, SparkFun-Capacitors:CAP0603-CAP
- removed J1, J12, J13, J2: (no value), i2c_encoder:M021X02_NO_SILK
- removed J3, J7: (no value), i2c_encoder:M04NO_SILK_ALL_ROUND
- removed JP1, JP2: (no value), pinhead_plus:PINHD-1X31X03_SMT
- removed JP5: (no value), pinhead_plus:PINHD-1X41X04_SMT
- removed LED1, LED10, LED11, LED12, LED13, LED14, LED15, LED16, LED17, LED18, LED19, LED2, LED3, LED31, LED32, LED33, LED34, LED35, LED36, LED37, LED38, LED39, LED4, LED40, LED41, LED42, LED43, LED44, LED45, LED5, LED6, LED7, LED8, LED9: WS2812B3535, i2c_encoder:WS2812B3535
- removed R1, R10, R11, R12, R13, R14, R15, R2, R3, R4, R41, R42, R43, R44, R45, R46, R47, R48, R49, R5, R50, R51, R52, R53, R54, R55, R6, R7, R8, R9: (no value), rcl:R-EU_R0603
- removed R26, R29, R30, R31: 0, rcl:R-EU_R0603
- removed R32, R33, R34, R35: 10k, rcl:R-EU_R0603
- removed S1: BUTTONPAD-2X2, i2c_encoder:BUTTONPAD-2X2
- removed SL1, SL2: (no value), con-amp-quick:M06
- removed U$1: 6PIN_1.27MM_POGO, i2c_encoder:6PIN_1.27MM_POGO
- removed X5: 52745-0690, i2c_encoder:52745-0690
Connections:
- removed net N$1: LED10.DO, LED11.DI, R12.2, R13.1
- removed net N$10: LED8.DO, LED9.DI, R10.2, R11.1
- removed net N$11: LED3.DO, LED4.DI, R5.2, R6.1
- removed net N$12: LED14.DO, LED15.DI, R1.2, R2.1
- removed net N$13: LED16.DO, LED18.DI, R26.1, R30.1
- removed net N$14: LED1.DO, LED2.DI, R3.2, R4.1
- removed net N$16: LED42.DO, LED43.DI, R46.2, R47.1
- removed net N$17: LED4.DO, LED5.DI, R6.2, R7.1
- removed net N$18: LED5.DO, LED6.DI, R7.2, R8.1
- removed net N$19: LED6.DO, LED7.DI, R8.2, R9.1
- removed net N$2: LED11.DO, LED12.DI, R13.2, R14.1
- removed net N$20: LED43.DO, LED44.DI, R47.2, R48.1
- removed net N$21: LED44.DO, LED45.DI, R48.2, R49.1
- removed net N$22: LED10.DI, LED9.DO, R11.2, R12.1
- removed net N$23: LED32.DO, LED33.DI, R51.2, R52.1
- removed net N$24: LED33.DO, LED34.DI, R52.2, R53.1
- removed net N$25: LED34.DO, LED35.DI, R53.2, R54.1
- removed net N$26: LED35.DO, LED36.DI, R54.2, R55.1
- removed net N$27: LED7.DO, LED8.DI, R10.1, R9.2
- removed net N$28: LED31.DO, LED32.DI, R50.2, R51.1
- removed net N$29: LED40.DO, LED41.DI, R44.2, R45.1
- removed net N$3: LED37.DO, LED38.DI, R41.2, R42.1
- removed net N$30: LED41.DO, LED42.DI, R45.2, R46.1
- removed net N$4: LED38.DO, LED39.DI, R42.2, R43.1
- removed net N$43: LED17.DI, LED19.DO, R29.2, R31.1
- removed net N$44: LED18.DO, LED19.DI, R26.2, R29.1
- removed net N$46: LED36.DO, LED37.DI, R41.1, R55.2
- removed net N$5: LED2.DO, LED3.DI, R4.2, R5.1
- removed net N$6: LED13.DO, LED14.DI, R1.1, R15.2
- removed net N$8: LED39.DO, LED40.DI, R43.2, R44.1
- removed net N$9: LED12.DO, LED13.DI, R14.2, R15.1
- removed net RST: SL1.1, U$1.1
- net !SS: no longer SL2.4, X5-4.S
- net ENC1A: now also IC1.PD2(INT0); no longer IC1.PD0(RXD), JP2.1, R33.1, S1C4.SIG1, SH1.P$1
- net ENC1B: now also IC1.PD3(INT1); no longer IC1.PC3(ADC3), JP2.3, R32.1, S1C3.SIG1
- net ENCL1A: now also IC1.PC3(ADC3); no longer IC1.PD3(INT1)
- net ENCL2A: now also IC1.PD0(RXD), SH1.P$1; no longer IC1.PD2(INT0)
- net ENC_SW: no longer JP1.1, R35.1, S1C2.SIG1
- net GND: no longer C1.2, C10.2, C11.2, C12.2, C13.2, C14.2, C15.2, C2.2, C20.2, C21.2, C22.2, C24.2, C3.2, C4.2, C41.2, C42.2, C43.2, C44.2, C45.2, C46.2, C47.2, C48.2, C49.2, C5.2, C50.2, C51.2, C52.2, C53.2, C54.2, C55.2, C6.2, C7.2, C8.2, C9.2, J1.2, J12.2, J13.2, J2.2, J3.4, J7.4, JP1.3, JP2.2, JP5.4, LED1.GND, LED10.GND, LED11.GND, LED12.GND, LED13.GND, LED14.GND, LED15.GND, LED16.GND, LED17.GND, LED18.GND, LED19.GND, LED2.GND, LED3.GND, LED31.GND, LED32.GND, LED33.GND, LED34.GND, LED35.GND, LED36.GND, LED37.GND, LED38.GND, LED39.GND, LED4.GND, LED40.GND, LED41.GND, LED42.GND, LED43.GND, LED44.GND, LED45.GND, LED5.GND, LED6.GND, LED7.GND, LED8.GND, LED9.GND, S1C1.SIG2, S1C2.SIG2, S1C3.SIG2, S1C4.SIG2, SL1.5, U$1.5
- net LED1: no longer J3.3, J7.3, JP5.3, LED1.DI, LED16.DI, LED31.DI, R3.1, R30.2, R50.1
- net LED_OUT: no longer J3.2, J7.2, JP5.2, LED15.DO, LED17.DO, LED45.DO, R2.2, R31.2, R49.2
- net MISO: no longer SL1.3, SL2.2, U$1.3, X5-2.S
- net MOSI: no longer SL1.2, SL2.3, U$1.2, X5-3.S
- net POT: no longer JP1.2, R34.1, S1C1.SIG1
- net SCK: no longer SL1.4, SL2.1, U$1.4, X5-1.S
- net SCL: no longer SL2.5, X5-5.S
- net SDA: no longer SL2.6, X5-6.S
- net VCC: no longer C1.1, C10.1, C11.1, C12.1, C13.1, C14.1, C15.1, C2.1, C20.1, C21.1, C22.1, C24.1, C3.1, C4.1, C41.1, C42.1, C43.1, C44.1, C45.1, C46.1, C47.1, C48.1, C49.1, C5.1, C50.1, C51.1, C52.1, C53.1, C54.1, C55.1, C6.1, C7.1, C8.1, C9.1, J1.1, J12.1, J13.1, J2.1, J3.1, J7.1, JP5.1, LED1.VDD, LED10.VDD, LED11.VDD, LED12.VDD, LED13.VDD, LED14.VDD, LED15.VDD, LED16.VDD, LED17.VDD, LED18.VDD, LED19.VDD, LED2.VDD, LED3.VDD, LED31.VDD, LED32.VDD, LED33.VDD, LED34.VDD, LED35.VDD, LED36.VDD, LED37.VDD, LED38.VDD, LED39.VDD, LED4.VDD, LED40.VDD, LED41.VDD, LED42.VDD, LED43.VDD, LED44.VDD, LED45.VDD, LED5.VDD, LED6.VDD, LED7.VDD, LED8.VDD, LED9.VDD, R32.2, R33.2, R34.2, R35.2, SL1.6, U$1.6
Other:
- note removed: "Adapter boards"
