File: eagle/connector_board.brd (EAGLE design)
At the start: 22.6 x 24.3 mm, 22 parts, among them IC1 MEGA8-MI, J1 FH12-6S-0.5SH(55), J2 FH12-6S-0.5SH(55), J3 FH12-6S-0.5SH(55), J4 FH12-6S-0.5SH(55), X4 POGOPIN-CONNWITHVIAS-SMV, X6 POGOPIN-CONNWITHVIAS-SMV

Commit message: Board version 4 WIP;
* Added solder pads to FFC connectors
* Fixed naming of connectors (previously M was on the right and labels
  were wrong
* Flipped builtin led (D1) around to make it safer to use with encoders
Parts:
- added U$1, U$2, U$3, U$4: 6PIN_SOLDER_PAD, edge:6PIN_SOLDER_PAD
- moved R40 2.77 mm to (19.1, 11.6), turned to 45 degrees
- moved D1 2.32 mm to (20.3, 14.0)
Connections:
- net !SS: now also U$4.P$4
- net ENCL1A: now also U$3.P$6
- net ENCL1B: now also U$3.P$5
- net ENCL2A: now also U$3.P$3
- net ENCL2B: now also U$3.P$2
- net ENCM1A: now also IC1.9, J3.1, U$1.P$6; no longer IC1.32, J4.1
- net ENCM1B: now also IC1.10, J3.2, U$1.P$5; no longer IC1.1, J4.2
- net ENCM2A: now also IC1.12, J3.4, U$1.P$3; no longer IC1.7, J4.4
- net ENCM2B: now also D1.-, IC1.13, J3.5, U$1.P$2; no longer IC1.8, J4.5
- net ENCR1A: now also IC1.32, J4.1, U$2.P$6; no longer IC1.9, J3.1
- net ENCR1B: now also IC1.1, J4.2, U$2.P$5; no longer IC1.10, J3.2
- net ENCR2A: now also IC1.7, J4.4, U$2.P$3; no longer IC1.12, J3.4
- net ENCR2B: now also IC1.8, J4.5, U$2.P$2; no longer D1.-, IC1.13, J3.5
- net GND: no longer R40.1
- net LEDL: now also U$3.P$4
- net LEDM: now also IC1.11, J3.3, U$1.P$4; no longer IC1.2, J4.3
- net LEDR: now also IC1.2, J4.3, U$2.P$4; no longer IC1.11, J3.3
- net MISO: now also U$4.P$2
- net MOSI: now also U$4.P$3
- net SCK: now also U$4.P$1
- net SCL: now also U$4.P$5
- net SDA: now also U$4.P$6
- net SWL: now also U$3.P$1
- net SWM: now also IC1.19, J3.6, U$1.P$1; no longer IC1.26, J4.6
- net SWR: now also IC1.26, J4.6, U$2.P$1; no longer IC1.19, J3.6
- net VCC: now also R40.1
Routing:
- net SWR: track 4.99 -> 20.4 mm, vias 2 -> 3
- net ENCR2A: track 1.57 -> 13.5 mm, vias 0 -> 1
- net ENCR1A: track 1.57 -> 11.1 mm, vias 0 -> 1
- net ENCR1B: track 1.57 -> 10.5 mm, vias 0 -> 1
- net LEDR: track 1.57 -> 10.4 mm, vias 0 -> 1
- net ENCM2B: track 8.21 -> 15.7 mm, vias 0 -> 2
- net SWL: track 8.00 -> 14.7 mm, vias 0 -> 2
- net SDA: track 6.40 -> 12.5 mm, vias 0 -> 1
- net ENCL1A: track 3.62 -> 9.50 mm, vias 0 -> 1
- net SCK: track 27.1 -> 32.8 mm, vias 3 -> 4
- net SCL: track 6.64 -> 12.2 mm, vias 0 -> 1
- net ENCL2B: track 18.6 -> 24.2 mm, vias 2 -> 3
- net ENCL1B: track 3.57 -> 9.13 mm, vias 0 -> 1
- net ENCR2B: track 7.82 -> 13.3 mm, vias 2 -> 1
- net !SS: track 17.0 -> 22.4 mm, vias 2 -> 3
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